Commit message: fix bug for remain rrt_exploration_tutorials package
fix bug for remain rrt_exploration_tutorials package

File: launch/includes/urdf/kobuki.urdf.xacro (robot description, xacro)
@@ -7,6 +7,6 @@
  -->
 <robot name="kobuki" xmlns:xacro="http://ros.org/wiki/xacro">
-  <xacro:include filename="$(find rrt_exploration_tutorials)/launch/includes/urdf/common_properties.urdf.xacro"/>
-  <xacro:include filename="$(find rrt_exploration_tutorials)/launch/includes/urdf/kobuki_gazebo.urdf.xacro"/>
+  <xacro:include filename="$(find multi_slam_karto)/launch/includes/urdf/common_properties.urdf.xacro"/>
+  <xacro:include filename="$(find multi_slam_karto)/launch/includes/urdf/kobuki_gazebo.urdf.xacro"/>
   <!-- Kobuki -->
   <xacro:macro name="kobuki">
@@ -30,5 +30,5 @@
         <geometry>
           <!-- new mesh -->
-          <mesh filename="package://rrt_exploration_tutorials/launch/includes/meshes/main_body.dae" />
+          <mesh filename="package://multi_slam_karto/launch/includes/meshes/main_body.dae" />
         </geometry>
         <origin xyz="0.001 0 0.05199" rpy="0 0 0"/>
@@ -65,5 +65,5 @@
       <visual>
         <geometry>
-          <mesh filename="package://rrt_exploration_tutorials/launch/includes/meshes/wheel.dae"/>
+          <mesh filename="package://multi_slam_karto/launch/includes/meshes/wheel.dae"/>
         </geometry>
         <origin xyz="0 0 0" rpy="0 0 0"/>
@@ -92,5 +92,5 @@
       <visual>
         <geometry>
-          <mesh filename="package://rrt_exploration_tutorials/launch/includes/meshes/wheel.dae"/>
+          <mesh filename="package://multi_slam_karto/launch/includes/meshes/wheel.dae"/>
         </geometry>
         <origin xyz="0 0 0" rpy="0 0 0"/>
@@ -223,5 +223,5 @@
       <origin xyz="0 0 0" rpy="0 0 0"/>
       <geometry>
-        <mesh filename="package://rrt_exploration_tutorials/launch/includes/meshes/hokuyo.dae"/>
+        <mesh filename="package://multi_slam_karto/launch/includes/meshes/hokuyo.dae"/>
       </geometry>
     </visual>

File: launch/includes/urdf/kobuki_standalone.urdf.xacro (robot description, xacro)
@@ -6,5 +6,5 @@
        xmlns:xacro="http://ros.org/wiki/xacro">
   <!-- Defines the kobuki component tag. -->
-  <xacro:include filename="$(find rrt_exploration_tutorials)/launch/includes/urdf/kobuki.urdf.xacro" />
+  <xacro:include filename="$(find multi_slam_karto)/launch/includes/urdf/kobuki.urdf.xacro" />
   <kobuki/>
 </robot>
